File: AnalogPeripherial.kicad_sch (KiCad schematic)
At the start: 52 parts, among them J1 USART, J2 SWD, J3 USB_B_Mini, SW1 record, SW2 replay, SW3 SW_Nidec_CAS-120A1, U1 LD1117S33TR_SOT223, U2 STM32F373CCTx, U3 LM386, U4 112J-TDAR-R01, U5 TLV9061xDBV, Y1 Crystal

Commit message: PCB progress
Parts:
- removed U4: 112J-TDAR-R01, 112J_TDAR_R01:112J-TDAR-R01_ATT, symbol 2025-12-27_23-38-34:112J-TDAR-R01
- added U4: ~, my_custom_stuff:microSD, symbol my_custom_stuff:microSD
- Y1: footprint Crystal:Crystal_HC18-U_Vertical -> Crystal:Crystal_HC49-4H_Vertical
Connections:
- net 3V3: now also U4.4 (VDD)
- net ADC1_IN1: now also U2.11 (PA1); no longer U2.10 (PA0)
- net GND: now also U4.6 (VSS)
- net SPI1_MISO: now also U4.7 (DAT0)
- net SPI1_MOSI: now also U4.3 (CMD)
- net SPI1_NSS: now also U4.2 (CD)
- net SPI1_SCK: now also U4.5 (CLK)
- net USART_RX renamed USART1_RX
- net USART_TX renamed USART1_TX
- no-connect marks 27 -> 26
Other:
- moved on the sheet: D2, R3, R4, SW1
